File: pcb/R1002A.kicad_pcb (KiCad board)
At the start: 2 copper layers, 45 x 33.3 mm, 25 parts, among them J1 PCIEXPRESS-X1, J2 CONN_01X04, J3 CONN_01X04, Q1 Q_NMOS_GDSD, Q2 Q_NMOS_GDSD, Q3 Q_NMOS_GDSD, Q4 Q_NMOS_GDSD, U1 MC14504B-TSSOP, U2 EFM8BB10F2G

Commit message: releasing first beta
Parts:
- added G***: LOGO, pluggee:pluggee-QRNEG-085X085, B.Cu at (131.2, 81.3)
Other:
- board text added: "+"
- board text added: "-"
- board text added: "1"
- board text added: "2"
- board text added: "3"
- board text added: "4"
- board text added: "R1002 v1.0.0-beta 1A NFET Drivers http://plugg.ee"
- board text added: "plugg.ee Labs 2016"
