File: pcb/R1002.kicad_pcb (KiCad board)
At the start: 2 copper layers, 45 x 33.3 mm, 13 parts, among them J1 PCIEXPRESS-X1, J2 CONN254P-02X04, Q1 Q_NMOS_GDSD, Q2 Q_NMOS_GDSD, Q3 Q_NMOS_GDSD, Q4 Q_NMOS_GDSD, U1 MC14504B-TSSOP

Commit message: getting ready to release
Parts:
- moved FID2 6.00 mm to (173.9, 91.2)
- moved FID3 6.00 mm to (173.8, 72.0)
Other:
- board size 45 x 33.3 mm -> 51 x 33.3 mm
- board text added: "plugg.ee Labs LLC, USA R1002 v1.1.1, Quad 1A NFET Drivers Open Source Hardware (GPL v3.0) http://plugg.ee"
- board text removed: "plugg.ee Labs LLC, USA R1002 v1.1, Quad 1A NFET Drivers Open Source Hardware (GPL v3.0) http://plugg.ee"
Changed lines of the file:
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@@
     (links 86)
     (no_connects 0)
-    (area 124.924999 69.924999 170.075001 103.375001)
+    (area 124.924999 69.924999 176.075001 103.375001)
     (thickness 1.6)
     (drawings 39)
@@
   )
   (module Main:FIDTOP001 (layer B.Cu)
-    (at 167.9 91.2)
+    (at 173.9 91.2)
     (descr "Circular Fiducial, 1mm bare copper top; 2.54mm keepout")
     (tags marker)
@@
   )
   (module Main:FIDTOP001 (layer B.Cu)
-    (at 167.8 72)
+    (at 173.8 72)
     (descr "Circular Fiducial, 1mm bare copper top; 2.54mm keepout")
     (tags marker)
@@
       (solder_mask_margin 0.77) (clearance 0.77))
   )
+  (module Main:CAPC0603 (layer B.Cu)
+    (at 135 78.4 90)
+    (descr "Resistor SMD 0603, reflow soldering, Vishay (see dcrcw.pdf)")
+    (tags "resistor 0603")
+    (attr smd)
+    (fp_text reference C1 (at 0 1.27 90) (layer B.SilkS)
+      (effects (font (size 0.7 0.7) (thickness 0.15)) (justify mirror))
+    )
+    (fp_text value CC0603KRX7R9BB104 (at 0 -0.508 90) (layer B.Fab)
+      (effects (font (size 0.127 0.127) (thickness 0.03)) (justify mirror))
+    )
+    (fp_line (start -1.3 0.8) (end 1.3 0.8) (layer B.CrtYd) (width 0.05))
+    (fp_line (start -1.3 -0.8) (end 1.3 -0.8) (layer B.CrtYd) (width 0.05))
+    (fp_line (start -1.3 0.8) (end -1.3 -0.8) (layer B.CrtYd) (width 0.05))
+    (fp_line (start 1.3 0.8) (end 1.3 -0.8) (layer B.CrtYd) (width 0.05))
+    (fp_line (start 0.5 -0.675) (end -0.5 -0.675) (layer B.SilkS) (width 0.15))
+    (fp_line (start -0.5 0.675) (end 0.5 0.675) (layer B.SilkS) (width 0.15))
+    (pad 1 smd rect (at -0.7745 0 90) (size 0.787 0.864) (layers B.Cu B.Paste B.Mask)
+      (net 3 +3V3))
+    (pad 2 smd rect (at 0.7745 0 90) (size 0.787 0.864) (layers B.Cu B.Paste B.Mask)
+      (net 2 GND))
+    (model main.3dshapes/CAPC0603.wrl
+      (at (xyz 0 0 0))
+      (scale (xyz 1 1 1))
+      (rotate (xyz 0 0 0))
+    )
+  )
+  (module Main:CAPC0603 (layer B.Cu)
+    (at 129 78.4 90)
+    (descr "Resistor SMD 0603, reflow soldering, Vishay (see dcrcw.pdf)")
+    (tags "resistor 0603")
+    (attr smd)
+    (fp_text reference C3 (at 0 1.27 90) (layer B.SilkS)
+      (effects (font (size 0.7 0.7) (thickness 0.15)) (justify mirror))
+    )
+    (fp_text value CC0603KRX7R9BB104 (at 0 -0.508 90) (layer B.Fab)
+      (effects (font (size 0.127 0.127) (thickness 0.03)) (justify mirror))
+    )
+    (fp_line (start -1.3 0.8) (end 1.3 0.8) (layer B.CrtYd) (width 0.05))
+    (fp_line (start -1.3 -0.8) (end 1.3 -0.8) (layer B.CrtYd) (width 0.05))
+    (fp_line (start -1.3 0.8) (end -1.3 -0.8) (layer B.CrtYd) (width 0.05))
+    (fp_line (start 1.3 0.8) (end 1.3 -0.8) (layer B.CrtYd) (width 0.05))
+    (fp_line (start 0.5 -0.675) (end -0.5 -0.675) (layer B.SilkS) (width 0.15))
+    (fp_line (start -0.5 0.675) (end 0.5 0.675) (layer B.SilkS) (width 0.15))
+    (pad 1 smd rect (at -0.7745 0 90) (size 0.787 0.864) (layers B.Cu B.Paste B.Mask)
+      (net 10 +5V))
+    (pad 2 smd rect (at 0.7745 0 90) (size 0.787 0.864) (layers B.Cu B.Paste B.Mask)
+      (net 2 GND))
+    (model main.3dshapes/CAPC0603.wrl
+      (at (xyz 0 0 0))
+      (scale (xyz 1 1 1))
+      (rotate (xyz 0 0 0))
+    )
+  )
   (module Main:CONN254P-02X04 (layer B.Cu)
     (at 166.3 82 90)
     (descr "Through hole socket strip")
     (tags "socket strip")
-    (fp_text reference J2 (at 9 -2.6 90) (layer B.SilkS)
+    (fp_text reference J2 (at 0 3.81 90) (layer B.SilkS) hide
       (effects (font (size 1 1) (thickness 0.15)) (justify mirror))
     )
@@
       (net 22 /DN1))
     (model main.3dshapes/CONN254P-02X04.wrl
-      (at (xyz -0.15 0 0))
-      (scale (xyz 0.3937 0.3937 0.3937))
-      (rotate (xyz -90 0 180))
-    )
-  )
-  (module Main:CAPC0603 (layer B.Cu)
-    (at 135 78.4 90)
-    (descr "Resistor SMD 0603, reflow soldering, Vishay (see dcrcw.pdf)")
-    (tags "resistor 0603")
-    (attr smd)
-    (fp_text reference C1 (at 0 1.27 90) (layer B.SilkS)
-      (effects (font (size 0.7 0.7) (thickness 0.15)) (justify mirror))
-    )
-    (fp_text value CC0603KRX7R9BB104 (at 0 -0.508 90) (layer B.Fab)
-      (effects (font (size 0.127 0.127) (thickness 0.03)) (justify mirror))
-    )
-    (fp_line (start -1.3 0.8) (end 1.3 0.8) (layer B.CrtYd) (width 0.05))
-    (fp_line (start -1.3 -0.8) (end 1.3 -0.8) (layer B.CrtYd) (width 0.05))
-    (fp_line (start -1.3 0.8) (end -1.3 -0.8) (layer B.CrtYd) (width 0.05))
-    (fp_line (start 1.3 0.8) (end 1.3 -0.8) (layer B.CrtYd) (width 0.05))
-    (fp_line (start 0.5 -0.675) (end -0.5 -0.675) (layer B.SilkS) (width 0.15))
-    (fp_line (start -0.5 0.675) (end 0.5 0.675) (layer B.SilkS) (width 0.15))
-    (pad 1 smd rect (at -0.7745 0 90) (size 0.787 0.864) (layers B.Cu B.Paste B.Mask)
-      (net 3 +3V3))
-    (pad 2 smd rect (at 0.7745 0 90) (size 0.787 0.864) (layers B.Cu B.Paste B.Mask)
-      (net 2 GND))
-    (model main.3dshapes/CAPC0603.wrl
       (at (xyz 0 0 0))
       (scale (xyz 1 1 1))
@@
     )
   )
-  (module Main:CAPC0603 (layer B.Cu)
-    (at 129 78.4 90)
-    (descr "Resistor SMD 0603, reflow soldering, Vishay (see dcrcw.pdf)")
-    (tags "resistor 0603")
-    (attr smd)
-    (fp_text reference C3 (at 0 1.27 90) (layer B.SilkS)
-      (effects (font (size 0.7 0.7) (thickness 0.15)) (justify mirror))
-    )
-    (fp_text value CC0603KRX7R9BB104 (at 0 -0.508 90) (layer B.Fab)
-      (effects (font (size 0.127 0.127) (thickness 0.03)) (justify mirror))
-    )
-    (fp_line (start -1.3 0.8) (end 1.3 0.8) (layer B.CrtYd) (width 0.05))
-    (fp_line (start -1.3 -0.8) (end 1.3 -0.8) (layer B.CrtYd) (width 0.05))
-    (fp_line (start -1.3 0.8) (end -1.3 -0.8) (layer B.CrtYd) (width 0.05))
-    (fp_line (start 1.3 0.8) (end 1.3 -0.8) (layer B.CrtYd) (width 0.05))
-    (fp_line (start 0.5 -0.675) (end -0.5 -0.675) (layer B.SilkS) (width 0.15))
-    (fp_line (start -0.5 0.675) (end 0.5 0.675) (layer B.SilkS) (width 0.15))
-    (pad 1 smd rect (at -0.7745 0 90) (size 0.787 0.864) (layers B.Cu B.Paste B.Mask)
-      (net 10 +5V))
-    (pad 2 smd rect (at 0.7745 0 90) (size 0.787 0.864) (layers B.Cu B.Paste B.Mask)
-      (net 2 GND))
-    (model main.3dshapes/CAPC0603.wrl
-      (at (xyz 0 0 0))
-      (scale (xyz 1 1 1))
-      (rotate (xyz 0 0 0))
-    )
-  )
   (gr_text 4 (at 162.1 85.8 90) (layer B.SilkS)
     (effects (font (size 2 2) (thickness 0.2)) (justify mirror))
@@
     (effects (font (size 2 2) (thickness 0.2)) (justify mirror))
   )
-  (gr_text 4 (at 162.1 85.9 90) (layer F.SilkS)
+  (gr_text 4 (at 172.1 85.9 90) (layer F.SilkS)
     (effects (font (size 2 2) (thickness 0.2)))
   )
-  (gr_text 3 (at 162.1 83.3 90) (layer F.SilkS)
+  (gr_text 3 (at 172.1 83.3 90) (layer F.SilkS)
     (effects (font (size 2 2) (thickness 0.2)))
   )
-  (gr_text 2 (at 162.1 80.6 90) (layer F.SilkS)
+  (gr_text 2 (at 172.1 80.6 90) (layer F.SilkS)
     (effects (font (size 2 2) (thickness 0.2)))
   )
-  (gr_text 1 (at 162.1 78.2 90) (layer F.SilkS)
+  (gr_text 1 (at 172.1 78.2 90) (layer F.SilkS)
     (effects (font (size 2 2) (thickness 0.2)))
   )
@@
     (effects (font (size 2 2) (thickness 0.2)) (justify mirror))
   )
-  (gr_text "plugg.ee Labs LLC, USA\nR1002 v1.1, Quad 1A NFET Drivers\nOpen Source Hardware (GPL v3.0)\nhttp://plugg.ee" (at 126.75 84.5) (layer F.SilkS)
+  (gr_text "plugg.ee Labs LLC, USA\nR1002 v1.1.1, Quad 1A NFET Drivers\nOpen Source Hardware (GPL v3.0)\nhttp://plugg.ee" (at 126.75 84.5) (layer F.SilkS)
     (effects (font (size 1 1) (thickness 0.2)) (justify left))
   )
-  (gr_arc (start 169.6 70.4) (end 170 70.4) (angle -90) (layer Edge.Cuts) (width 0.15))
-  (gr_arc (start 169.6 93.1) (end 169.6 93.5) (angle -90) (layer Edge.Cuts) (width 0.15))
+  (gr_arc (start 175.6 70.4) (end 176 70.4) (angle -90) (layer Edge.Cuts) (width 0.15))
+  (gr_arc (start 175.6 93.1) (end 175.6 93.5) (angle -90) (layer Edge.Cuts) (width 0.15))
   (gr_arc (start 159.75 102.9) (end 160.15 102.9) (angle 90) (layer Edge.Cuts) (width 0.15))
   (gr_arc (start 149.35 102.9) (end 148.95 102.9) (angle -90) (layer Edge.Cuts) (width 0.15))
   (gr_arc (start 146.65 102.9) (end 147.05 102.9) (angle 90) (layer Edge.Cuts) (width 0.15))
   (gr_arc (start 140.25 102.9) (end 139.85 102.9) (angle -90) (layer Edge.Cuts) (width 0.15))
-  (gr_line (start 170 70.4) (end 170 93.1) (angle 90) (layer Edge.Cuts) (width 0.15))
-  (gr_line (start 169.6 93.5) (end 161.1 93.5) (angle 90) (layer Edge.Cuts) (width 0.15))
+  (gr_line (start 176 70.4) (end 176 93.1) (angle 90) (layer Edge.Cuts) (width 0.15))
+  (gr_line (start 175.6 93.5) (end 161.1 93.5) (angle 90) (layer Edge.Cuts) (width 0.15))
   (gr_arc (start 161.1 94.45) (end 160.15 94.45) (angle 90) (layer Edge.Cuts) (width 0.15))
   (gr_line (start 125 91.5) (end 125 72) (angle 90) (layer Edge.Cuts) (width 0.15))
@@
   (gr_arc (start 138.9 94.45) (end 139.85 94.45) (angle -90) (layer Edge.Cuts) (width 0.15))
   (gr_arc (start 127 72) (end 125 72) (angle 90) (layer Edge.Cuts) (width 0.15))
-  (gr_line (start 169.6 70) (end 127 70) (angle 90) (layer Edge.Cuts) (width 0.15))
+  (gr_line (start 175.6 70) (end 127 70) (angle 90) (layer Edge.Cuts) (width 0.15))
   (gr_line (start 160.15 102.9) (end 160.15 94.45) (angle 90) (layer Edge.Cuts) (width 0.15))
   (gr_line (start 149.35 103.3) (end 159.75 103.3) (angle 90) (layer Edge.Cuts) (width 0.15))
@@
     (polygon
       (pts
-        (xy 171 105) (xy 124 105) (xy 124 69) (xy 171 69)
+        (xy 180.7 105) (xy 124 105) (xy 124 69) (xy 180.7 69)
       )
     )
@@
     (polygon
       (pts
-        (xy 152.175 100.45) (xy 152.175 90.5) (xy 166.45 90.5) (xy 166.575 90.375) (xy 166.575 73.75)
-        (xy 169.675 73.725) (xy 169.675 93.125) (xy 159.8 93.125) (xy 159.8 100.45)
+        (xy 152.175 100.45) (xy 152.175 90.5) (xy 166.45 90.5) (xy 166.575 90.375) (xy 166.6 67.5)
+        (xy 177.8 67.5) (xy 177.8 93.1) (xy 159.8 93.125) (xy 159.8 100.45)
       )
     )

Commit message: narrowed PCB to avoid connector bump into PCB
Parts:
- moved FID2 4.00 mm to (169.9, 91.2)
- moved FID3 4.00 mm to (169.8, 72.0)
Other:
- board size 51 x 33.3 mm -> 47 x 33.3 mm
Changed lines of the file:
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@@
     (links 86)
     (no_connects 0)
-    (area 124.924999 69.924999 176.075001 103.375001)
+    (area 124.924999 69.924999 172.075001 103.375001)
     (thickness 1.6)
     (drawings 39)
@@
   )
   (module Main:FIDTOP001 (layer B.Cu)
-    (at 173.9 91.2)
+    (at 169.9 91.2)
     (descr "Circular Fiducial, 1mm bare copper top; 2.54mm keepout")
     (tags marker)
@@
   )
   (module Main:FIDTOP001 (layer B.Cu)
-    (at 173.8 72)
+    (at 169.8 72)
     (descr "Circular Fiducial, 1mm bare copper top; 2.54mm keepout")
     (tags marker)
@@
     (effects (font (size 2 2) (thickness 0.2)) (justify mirror))
   )
-  (gr_text 4 (at 172.1 85.9 90) (layer F.SilkS)
+  (gr_text 4 (at 170.5 85.9 90) (layer F.SilkS)
     (effects (font (size 2 2) (thickness 0.2)))
   )
-  (gr_text 3 (at 172.1 83.3 90) (layer F.SilkS)
+  (gr_text 3 (at 170.5 83.3 90) (layer F.SilkS)
     (effects (font (size 2 2) (thickness 0.2)))
   )
-  (gr_text 2 (at 172.1 80.6 90) (layer F.SilkS)
+  (gr_text 2 (at 170.5 80.6 90) (layer F.SilkS)
     (effects (font (size 2 2) (thickness 0.2)))
   )
-  (gr_text 1 (at 172.1 78.2 90) (layer F.SilkS)
+  (gr_text 1 (at 170.5 78.2 90) (layer F.SilkS)
     (effects (font (size 2 2) (thickness 0.2)))
   )
@@
     (effects (font (size 1 1) (thickness 0.2)) (justify left))
   )
-  (gr_arc (start 175.6 70.4) (end 176 70.4) (angle -90) (layer Edge.Cuts) (width 0.15))
-  (gr_arc (start 175.6 93.1) (end 175.6 93.5) (angle -90) (layer Edge.Cuts) (width 0.15))
+  (gr_arc (start 171.6 70.4) (end 172 70.4) (angle -90) (layer Edge.Cuts) (width 0.15))
+  (gr_arc (start 171.6 93.1) (end 171.6 93.5) (angle -90) (layer Edge.Cuts) (width 0.15))
   (gr_arc (start 159.75 102.9) (end 160.15 102.9) (angle 90) (layer Edge.Cuts) (width 0.15))
   (gr_arc (start 149.35 102.9) (end 148.95 102.9) (angle -90) (layer Edge.Cuts) (width 0.15))
   (gr_arc (start 146.65 102.9) (end 147.05 102.9) (angle 90) (layer Edge.Cuts) (width 0.15))
   (gr_arc (start 140.25 102.9) (end 139.85 102.9) (angle -90) (layer Edge.Cuts) (width 0.15))
-  (gr_line (start 176 70.4) (end 176 93.1) (angle 90) (layer Edge.Cuts) (width 0.15))
-  (gr_line (start 175.6 93.5) (end 161.1 93.5) (angle 90) (layer Edge.Cuts) (width 0.15))
+  (gr_line (start 172 70.4) (end 172 93.1) (angle 90) (layer Edge.Cuts) (width 0.15))
+  (gr_line (start 171.6 93.5) (end 161.1 93.5) (angle 90) (layer Edge.Cuts) (width 0.15))
   (gr_arc (start 161.1 94.45) (end 160.15 94.45) (angle 90) (layer Edge.Cuts) (width 0.15))
   (gr_line (start 125 91.5) (end 125 72) (angle 90) (layer Edge.Cuts) (width 0.15))
@@
   (gr_arc (start 138.9 94.45) (end 139.85 94.45) (angle -90) (layer Edge.Cuts) (width 0.15))
   (gr_arc (start 127 72) (end 125 72) (angle 90) (layer Edge.Cuts) (width 0.15))
-  (gr_line (start 175.6 70) (end 127 70) (angle 90) (layer Edge.Cuts) (width 0.15))
+  (gr_line (start 171.6 70) (end 127 70) (angle 90) (layer Edge.Cuts) (width 0.15))
   (gr_line (start 160.15 102.9) (end 160.15 94.45) (angle 90) (layer Edge.Cuts) (width 0.15))
   (gr_line (start 149.35 103.3) (end 159.75 103.3) (angle 90) (layer Edge.Cuts) (width 0.15))
